Commit message: added a few links to the robot

File: src/robot_arm/urdf/robot_arm.urdf.xacro (robot description, xacro)
@@ -4,4 +4,10 @@
     <xacro:property name="base_width" value="0.1" />
     <xacro:property name="base_height" value="0.05" />
+    <xacro:property name="base_radius" value="0.05" />
+    <xacro:property name="base_depth" value="0.03" />
+    <xacro:property name="arm_radius" value="0.02" />
+    <xacro:property name="arm_depth" value="0.1" />
+    <xacro:property name="gripper_radius" value="0.04" />
+    <xacro:property name="gripper_length" value="0.05" />
     <link name="base_link">
         <visual>
@@ -12,3 +18,27 @@
         </visual>
     </link>
+    <link name="base2_link">
+        <visual>
+            <geometry>
+                <cylinder size="${base_radius} ${base_depth}" />
+            </geometry>
+            <origin xyz="0 0 0" rpy="0 0 0" />
+        </visual>
+    </link>
+    <link name="arm_link">
+        <visual>
+            <geometry>
+                <cylinder size="${arm_radius} ${arm_depth}" />
+            </geometry>
+            <origin xyz="0 0 0" rpy="0 0 0" />
+        </visual>
+    </link>
+    <link name="gripper_link">
+        <visual>
+            <geometry>
+                <cone size="${gripper_radius} ${gripper_length}" />
+            </geometry>
+            <origin xyz="0 0 0" rpy="0 0 0" />
+        </visual>
+    </link>
 </robot>

Commit message: I've included in joint links

File: src/robot_arm/urdf/robot_arm.urdf.xacro (robot description, xacro)
@@ -42,3 +42,18 @@
         </visual>
     </link>
+    <joint name="base_base2_joint" type="fixed">
+        <parent link="base_link" />
+        <child link="base2_link" />
+        <origin xyz="0 0 0" rpy="0 0 0" />
+    </joint>
+    <joint name="base2_arm_joint" type="revolute">
+        <parent link="base2_link" />
+        <child link="arm_link" />
+        <origin xyz="0 0 0" rpy="0 0 0" />
+    </joint>
+    <joint name="arm_gripper_joint" type="fixed">
+        <parent link="arm_link" />
+        <child link="gripper_link" />
+        <origin xyz="0 0 0" rpy="0 0 0" />
+    </joint>
 </robot>
