Commit message: Visualized my robotic arm in rviz2

File: install/robot_arm/share/robot_arm/urdf/robot_arm.urdf.xacro (robot description, xacro)
@@ -10,4 +10,5 @@
     <xacro:property name="gripper_radius" value="0.04" />
     <xacro:property name="gripper_length" value="0.05" />
+    <link name="base_footprint" />
     <link name="base_link">
         <visual>
@@ -21,5 +22,5 @@
         <visual>
             <geometry>
-                <cylinder size="${base_radius} ${base_depth}" />
+                <cylinder radius="${base_radius}" length="${base_depth}" />
             </geometry>
             <origin xyz="0 0 0" rpy="0 0 0" />
@@ -29,5 +30,5 @@
         <visual>
             <geometry>
-                <cylinder size="${arm_radius} ${arm_depth}" />
+                <cylinder radius="${arm_radius}" length="${arm_depth}" />
             </geometry>
             <origin xyz="0 0 0" rpy="0 0 0" />
@@ -37,9 +38,14 @@
         <visual>
             <geometry>
-                <cone size="${gripper_radius} ${gripper_length}" />
+                <cylinder radius="${gripper_radius}" length="${gripper_length}" />
             </geometry>
             <origin xyz="0 0 0" rpy="0 0 0" />
         </visual>
     </link>
+    <joint name="base_joint" type="fixed">
+        <parent link="base_footprint" />
+        <child link="base_link" />
+        <origin xyz="0 0 0" rpy="0 0 0" />
+    </joint>
     <joint name="base_base2_joint" type="fixed">
         <parent link="base_link" />
@@ -51,9 +57,12 @@
         <child link="arm_link" />
         <origin xyz="0 0 0" rpy="0 0 0" />
+        <axis xyz="0 0 1" />
+        <limit lower="-3.14" uppper="3.14" velocity="2.0" effort="200" />
     </joint>
-    <joint name="arm_gripper_joint" type="fixed">
+    <joint name="arm_gripper_joint" type="continuous">
         <parent link="arm_link" />
         <child link="gripper_link" />
         <origin xyz="0 0 0" rpy="0 0 0" />
+        <axis xyz="0 1 0" />
     </joint>
 </robot>

Commit message: added different material types

File: install/robot_arm/share/robot_arm/urdf/robot_arm.urdf.xacro (robot description, xacro)
@@ -10,4 +10,16 @@
     <xacro:property name="gripper_radius" value="0.04" />
     <xacro:property name="gripper_length" value="0.05" />
+    <material name="grey">
+        <color rgba="0.7 0.4 0 1" />
+    </material>
+    <material name="blue">
+        <color rgba="0 0 0.7 1" />
+    </material>
+    <material name="green">
+        <color rgba="0 1 0 1" />
+    </material>
+    <material name="red">
+        <color rgba="1 0 0 1" />
+    </material>
     <link name="base_footprint" />
     <link name="base_link">
@@ -17,4 +29,5 @@
             </geometry>
             <origin xyz="0 0 0" rpy="0 0 0" />
+            <material name="grey" />
         </visual>
     </link>
@@ -25,4 +38,5 @@
             </geometry>
             <origin xyz="0 0 0" rpy="0 0 0" />
+            <material name="red" />
         </visual>
     </link>
@@ -33,4 +47,5 @@
             </geometry>
             <origin xyz="0 0 0" rpy="0 0 0" />
+            <material name="green" />
         </visual>
     </link>
@@ -41,4 +56,5 @@
             </geometry>
             <origin xyz="0 0 0" rpy="0 0 0" />
+            <material name="blue" />
         </visual>
     </link>
@@ -47,4 +63,5 @@
         <child link="base_link" />
         <origin xyz="0 0 0" rpy="0 0 0" />
+        <axis xyz="0 0 0" />
     </joint>
     <joint name="base_base2_joint" type="fixed">

Commit message: this is an updated model with all the joints in function and in test.

File: install/robot_arm/share/robot_arm/urdf/robot_arm.urdf.xacro (robot description, xacro)
@@ -3,5 +3,5 @@
     <xacro:property name="base_length" value="0.1" />
     <xacro:property name="base_width" value="0.1" />
-    <xacro:property name="base_height" value="0.05" />
+    <xacro:property name="base_height" value="0.01" />
     <xacro:property name="base_radius" value="0.05" />
     <xacro:property name="base_depth" value="0.03" />
@@ -11,5 +11,5 @@
     <xacro:property name="gripper_length" value="0.05" />
     <material name="grey">
-        <color rgba="0.7 0.4 0 1" />
+        <color rgba="0.62 0.62 0.62 1" />
     </material>
     <material name="blue">
@@ -68,17 +68,17 @@
         <parent link="base_link" />
         <child link="base2_link" />
-        <origin xyz="0 0 0" rpy="0 0 0" />
+        <origin xyz="0 0 ${(base_height / 2.0) +(base_depth / 2.0)}" rpy="0 0 0" />
     </joint>
     <joint name="base2_arm_joint" type="revolute">
         <parent link="base2_link" />
         <child link="arm_link" />
-        <origin xyz="0 0 0" rpy="0 0 0" />
+        <origin xyz="0 0 ${(base_depth/2.0) + (arm_depth/2.0)}" rpy="0 0 0" />
         <axis xyz="0 0 1" />
-        <limit lower="-3.14" uppper="3.14" velocity="2.0" effort="200" />
+        <limit lower="-3.14" upper="3.14" velocity="2.0" effort="200" />
     </joint>
     <joint name="arm_gripper_joint" type="continuous">
         <parent link="arm_link" />
         <child link="gripper_link" />
-        <origin xyz="0 0 0" rpy="0 0 0" />
+        <origin xyz="0 0 ${(arm_depth/2.0) + (gripper_length/2.0)}" rpy="0 0 0" />
         <axis xyz="0 1 0" />
     </joint>

Commit message: I've included gazebo launch file so as to visualize and simulate the robotic arm

File: install/robot_arm/share/robot_arm/urdf/robot_arm.urdf.xacro (robot description, xacro)
@@ -1,25 +1,14 @@
 <?xml version="1.0"?>
 <robot name="robot_arm" xmlns:xacro="http://www.ros.org/wiki/xacro">
-    <xacro:property name="base_length" value="0.1" />
-    <xacro:property name="base_width" value="0.1" />
-    <xacro:property name="base_height" value="0.01" />
-    <xacro:property name="base_radius" value="0.05" />
-    <xacro:property name="base_depth" value="0.03" />
-    <xacro:property name="arm_radius" value="0.02" />
+    <xacro:include filename="robot_prop.xacro" />
+    <xacro:property name="base_length" value="0.2" />
+    <xacro:property name="base_width" value="0.15" />
+    <xacro:property name="base_height" value="0.03" />
+    <xacro:property name="base_radius" value="0.08" />
+    <xacro:property name="base_depth" value="0.05" />
+    <xacro:property name="arm_radius" value="0.05" />
     <xacro:property name="arm_depth" value="0.1" />
-    <xacro:property name="gripper_radius" value="0.04" />
-    <xacro:property name="gripper_length" value="0.05" />
-    <material name="grey">
-        <color rgba="0.62 0.62 0.62 1" />
-    </material>
-    <material name="blue">
-        <color rgba="0 0 0.7 1" />
-    </material>
-    <material name="green">
-        <color rgba="0 1 0 1" />
-    </material>
-    <material name="red">
-        <color rgba="1 0 0 1" />
-    </material>
+    <xacro:property name="gripper_radius" value="0.025" />
+    <xacro:property name="gripper_length" value="0.04" />
     <link name="base_footprint" />
     <link name="base_link">
@@ -31,4 +20,12 @@
             <material name="grey" />
         </visual>
+        <collision>
+            <geometry>
+                <box size="${base_length} ${base_width} ${base_height}" />
+            </geometry>
+            <origin xyz="0 0 0" rpy="0 0 0" />
+        </collision>
+        <xacro:base_inertia m="0.5" l="${base_length}" w="${base_width}" h="${base_height}"
+                            xyz="0 0 0" rpy="0 0 0" />
     </link>
     <link name="base2_link">
@@ -40,4 +37,12 @@
             <material name="red" />
         </visual>
+        <collision>
+            <geometry>
+                <cylinder radius="${base_radius}" length="${base_depth}" />
+            </geometry>
+            <origin xyz="0 0 0" rpy="0 0 0" />
+        </collision>
+        <xacro:base2_inertia m="0.5" r="${base_radius}" h="${base_depth}"
+                             xyz="0 0 0" rpy="0 0 0" />
     </link>
     <link name="arm_link">
@@ -49,4 +54,12 @@
             <material name="green" />
         </visual>
+        <collision>
+            <geometry>
+                <cylinder radius="${arm_radius}" length="${arm_depth}" />
+            </geometry>
+            <origin xyz="0 0 0" rpy="0 0 0" />
+        </collision>
+        <xacro:arm_inertia m="0.5" r="${arm_radius}" h="${arm_depth}"
+                            xyz="0 0 0" rpy="0 0 0" />
     </link>
     <link name="gripper_link">
@@ -58,4 +71,12 @@
             <material name="blue" />
         </visual>
+        <collision>
+            <geometry>
+                <cylinder radius="${gripper_radius}" length="${gripper_length}" />
+            </geometry>
+            <origin xyz="0 0 0" rpy="0 0 0" />
+        </collision>
+        <xacro:gripper_inertia m="0.5" r="${gripper_radius}" h="${gripper_length}"
+                                xyz="0 0 0" rpy="0 0 0" />
     </link>
     <joint name="base_joint" type="fixed">
@@ -82,4 +103,29 @@
         <origin xyz="0 0 ${(arm_depth/2.0) + (gripper_length/2.0)}" rpy="0 0 0" />
         <axis xyz="0 1 0" />
+        <limit lower="-1.57" upper="1.57" velocity="2.0" effort="200" />
     </joint>
+    <!-- Gazebo ROS Control Plugin -->
+    <gazebo>
+        <plugin filename="libgazebo_ros2_control.so" name="gazebo_ros2_control">
+            <parameters>$(find robot_arm)/config/arm_controllers.yaml</parameters>
+        </plugin>
+    </gazebo>
+    <!-- ROS 2 Control Transmissions -->
+    <ros2_control name="robot_arm" type="system">
+        <hardware>
+            <plugin>gazebo_ros2_control/GazeboSystem</plugin>
+        </hardware>
+        <joint name="base2_arm_joint">
+            <command_interface name="position"/>
+            <command_interface name="velocity"/>
+            <state_interface name="position"/>
+            <state_interface name="velocity"/>
+        </joint>
+        <joint name="arm_gripper_joint">
+            <command_interface name="position"/>
+            <command_interface name="velocity"/>
+            <state_interface name="position"/>
+            <state_interface name="velocity"/>
+        </joint>
+    </ros2_control>
 </robot>

File: src/robot_arm/urdf/robot_arm.urdf.xacro (robot description, xacro)
@@ -2,25 +2,13 @@
 <robot name="robot_arm" xmlns:xacro="http://www.ros.org/wiki/xacro">
     <xacro:include filename="robot_prop.xacro" />
-    <xacro:property name="base_length" value="0.1" />
-    <xacro:property name="base_width" value="0.1" />
-    <xacro:property name="base_height" value="0.01" />
-    <xacro:property name="base_radius" value="0.05" />
-    <xacro:property name="base_depth" value="0.03" />
-    <xacro:property name="arm_radius" value="0.02" />
+    <xacro:property name="base_length" value="0.2" />
+    <xacro:property name="base_width" value="0.15" />
+    <xacro:property name="base_height" value="0.03" />
+    <xacro:property name="base_radius" value="0.08" />
+    <xacro:property name="base_depth" value="0.05" />
+    <xacro:property name="arm_radius" value="0.05" />
     <xacro:property name="arm_depth" value="0.1" />
-    <xacro:property name="gripper_radius" value="0.04" />
-    <xacro:property name="gripper_length" value="0.05" />
-    <material name="grey">
-        <color rgba="0.62 0.62 0.62 1" />
-    </material>
-    <material name="blue">
-        <color rgba="0 0 0.7 1" />
-    </material>
-    <material name="green">
-        <color rgba="0 1 0 1" />
-    </material>
-    <material name="red">
-        <color rgba="1 0 0 1" />
-    </material>
+    <xacro:property name="gripper_radius" value="0.025" />
+    <xacro:property name="gripper_length" value="0.04" />
     <link name="base_footprint" />
     <link name="base_link">
@@ -32,4 +20,12 @@
             <material name="grey" />
         </visual>
+        <collision>
+            <geometry>
+                <box size="${base_length} ${base_width} ${base_height}" />
+            </geometry>
+            <origin xyz="0 0 0" rpy="0 0 0" />
+        </collision>
+        <xacro:base_inertia m="0.5" l="${base_length}" w="${base_width}" h="${base_height}"
+                            xyz="0 0 0" rpy="0 0 0" />
     </link>
     <link name="base2_link">
@@ -41,4 +37,12 @@
             <material name="red" />
         </visual>
+        <collision>
+            <geometry>
+                <cylinder radius="${base_radius}" length="${base_depth}" />
+            </geometry>
+            <origin xyz="0 0 0" rpy="0 0 0" />
+        </collision>
+        <xacro:base2_inertia m="0.5" r="${base_radius}" h="${base_depth}"
+                             xyz="0 0 0" rpy="0 0 0" />
     </link>
     <link name="arm_link">
@@ -50,4 +54,12 @@
             <material name="green" />
         </visual>
+        <collision>
+            <geometry>
+                <cylinder radius="${arm_radius}" length="${arm_depth}" />
+            </geometry>
+            <origin xyz="0 0 0" rpy="0 0 0" />
+        </collision>
+        <xacro:arm_inertia m="0.5" r="${arm_radius}" h="${arm_depth}"
+                            xyz="0 0 0" rpy="0 0 0" />
     </link>
     <link name="gripper_link">
@@ -59,4 +71,12 @@
             <material name="blue" />
         </visual>
+        <collision>
+            <geometry>
+                <cylinder radius="${gripper_radius}" length="${gripper_length}" />
+            </geometry>
+            <origin xyz="0 0 0" rpy="0 0 0" />
+        </collision>
+        <xacro:gripper_inertia m="0.5" r="${gripper_radius}" h="${gripper_length}"
+                                xyz="0 0 0" rpy="0 0 0" />
     </link>
     <joint name="base_joint" type="fixed">
@@ -83,4 +103,29 @@
         <origin xyz="0 0 ${(arm_depth/2.0) + (gripper_length/2.0)}" rpy="0 0 0" />
         <axis xyz="0 1 0" />
+        <limit lower="-1.57" upper="1.57" velocity="2.0" effort="200" />
     </joint>
+    <!-- Gazebo ROS Control Plugin -->
+    <gazebo>
+        <plugin filename="libgazebo_ros2_control.so" name="gazebo_ros2_control">
+            <parameters>$(find robot_arm)/config/arm_controllers.yaml</parameters>
+        </plugin>
+    </gazebo>
+    <!-- ROS 2 Control Transmissions -->
+    <ros2_control name="robot_arm" type="system">
+        <hardware>
+            <plugin>gazebo_ros2_control/GazeboSystem</plugin>
+        </hardware>
+        <joint name="base2_arm_joint">
+            <command_interface name="position"/>
+            <command_interface name="velocity"/>
+            <state_interface name="position"/>
+            <state_interface name="velocity"/>
+        </joint>
+        <joint name="arm_gripper_joint">
+            <command_interface name="position"/>
+            <command_interface name="velocity"/>
+            <state_interface name="position"/>
+            <state_interface name="velocity"/>
+        </joint>
+    </ros2_control>
 </robot>
